File: keyboard-split-splay-5x3+2-pinky-cluster.kicad_pcb (KiCad board)
At the start: 2 copper layers, 289.8 x 97.8 mm, 80 parts, among them SW1 GENERIC_ELECTROMECHANICAL_PUS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, SW10 GENERIC_ELECTROMECHANICAL_PUS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, SW11 GENERIC_ELECTROMECHANICAL_PUS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, SW12 GENERIC_ELECTROMECHANICAL_PUS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, SW13 GENERIC_ELECTROMECHANICAL_PUS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, SW14 GENERIC_ELECTROMECHANICAL_PUS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, SW15 GENERIC_ELECTROMECHANICAL_PUS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, SW16 GENERIC_ELECTROMECHANICAL_PUS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, SW17 GENERIC_ELECTROMECHANICAL_PUS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, SW18 GENERIC_ELECTROMECHANICAL_PUS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, SW19 GENERIC_ELECTROMECHANICAL_PUS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, SW2 GENERIC_ELECTROMECHANICAL_PUS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, SW20 GENERIC_ELECTROMECHANICAL_PUS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, SW21 GENERIC_ELECTROMECHANICAL_PUS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, SW22 GENERIC_ELECTROMECHANICAL_PUS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, SW23 GENERIC_ELECTROMECHANICAL_PUS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, SW24 GENERIC_ELECTROMECHANICAL_PUS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, SW25 GENERIC_ELECTROMECHANICAL_PUS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, SW26 GENERIC_ELECTROMECHANICAL_PUS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, SW27 GENERIC_ELECTROMECHANICAL_PUS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, SW28 GENERIC_ELECTROMECHANICAL_PUS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, SW29 GENERIC_ELECTROMECHANICAL_PUS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, SW3 GENERIC_ELECTROMECHANICAL_PUS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, SW30 GENERIC_ELECTROMECHANICAL_PUS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, SW31 GENERIC_ELECTROMECHANICAL_PUS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, SW32 GENERIC_ELECTROMECHANICAL_PUS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, SW33 GENERIC_ELECTROMECHANICAL_PUS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, SW34 GENERIC_ELECTROMECHANICAL_PUS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, SW35 GENERIC_ELECTROMECHANICAL_PUS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, SW36 GENERIC_ELECTROMECHANICAL_PUS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, SW4 GENERIC_ELECTROMECHANICAL_PUS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, SW5 GENERIC_ELECTROMECHANICAL_PUS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, SW6 GENERIC_ELECTROMECHANICAL_PUS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, SW7 GENERIC_ELECTROMECHANICAL_PUS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, SW8 GENERIC_ELECTROMECHANICAL_PUS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, SW9 GENERIC_ELECTROMECHANICAL_PUS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, U1 XIAO-RP2040-DIP, U2 XIAO-RP2040-DIP

Commit message: Rev 1.1, fix diode footprints, add plate and base generation jobs, add mouse bites and some extra solder jumpers
Parts:
- added ?: , , F.Cu at (170.7, 126.7)
- added ?: , , F.Cu at (170.7, 128.5)
- added ?: , , F.Cu at (165.0, 126.7)
- added ?: , , F.Cu at (165.0, 128.5)
- added ?: , , F.Cu at (165.0, 130.3)
- added ?: , , F.Cu at (170.7, 130.3)
- added JP5: SolderJumper_2_Open, Jumper:SolderJumper-2_P1.3mm_Open_RoundedPad1.0x1.5mm, F.Cu at (174.3, 129.0)
- added JP6: SolderJumper_2_Open, Jumper:SolderJumper-2_P1.3mm_Open_RoundedPad1.0x1.5mm, F.Cu at (174.3, 126.5)
- added JP7: SolderJumper_2_Open, Jumper:SolderJumper-2_P1.3mm_Open_RoundedPad1.0x1.5mm, F.Cu at (174.3, 123.9)
- added JP8: SolderJumper_2_Open, Jumper:SolderJumper-2_P1.3mm_Open_RoundedPad1.0x1.5mm, F.Cu at (174.3, 131.5)
- added M2: MECHANICAL_HOLE_5MM, benri-projects:MECHANICAL_HOLE_5MM, F.Cu at (190.8, 155.0)
- added REF**: MECHANICAL_HOLE_1MM_PLATED, benri-projects:MECHANICAL_HOLE_1MM_PLATED, F.Cu at (165.0, 124.8)
- added REF**: MECHANICAL_HOLE_5MM, benri-projects:MECHANICAL_HOLE_5MM, F.Cu at (209.8, 108.5)
- added REF**: MouseBite-Part_2.0x2.0mm_inset_D0.5mm_P0.85mm_5h, Panelization:MouseBite-Part_2.0x2.0mm_inset_D0.5mm_P0.85mm_5h, F.Cu at (165.2, 142.6)
- added REF**: MECHANICAL_HOLE_5MM, benri-projects:MECHANICAL_HOLE_5MM, F.Cu at (248.0, 103.0)
- added REF**: MECHANICAL_MOUSEBITES_4x0.5MM, benri-projects:MECHANICAL_MOUSEBITES_4x0.5MM, F.Cu at (170.4, 159.6)
- added REF**: MECHANICAL_HOLE_5MM, benri-projects:MECHANICAL_HOLE_5MM, F.Cu at (144.8, 155.0)
- added REF**: MECHANICAL_HOLE_5MM, benri-projects:MECHANICAL_HOLE_5MM, F.Cu at (45.5, 129.2)
- added REF**: MouseBite-Part_2.0x2.0mm_inset_D0.5mm_P0.85mm_5h, Panelization:MouseBite-Part_2.0x2.0mm_inset_D0.5mm_P0.85mm_5h, F.Cu at (170.4, 142.6)
- added REF**: MECHANICAL_HOLE_5MM, benri-projects:MECHANICAL_HOLE_5MM, F.Cu at (290.1, 129.2)
- added REF**: MECHANICAL_HOLE_5MM, benri-projects:MECHANICAL_HOLE_5MM, F.Cu at (87.6, 103.0)
- added REF**: MECHANICAL_HOLE_5MM, benri-projects:MECHANICAL_HOLE_5MM, F.Cu at (125.8, 108.5)
- added REF**: MECHANICAL_HOLE_5MM, benri-projects:MECHANICAL_HOLE_5MM, F.Cu at (238.2, 143.0)
- added REF**: MECHANICAL_HOLE_1MM_PLATED, benri-projects:MECHANICAL_HOLE_1MM_PLATED, F.Cu at (170.7, 124.8)
- added REF**: MECHANICAL_HOLE_5MM, benri-projects:MECHANICAL_HOLE_5MM, F.Cu at (97.3, 143.0)
- added REF**: MECHANICAL_MOUSEBITES_4x0.5MM, benri-projects:MECHANICAL_MOUSEBITES_4x0.5MM, F.Cu at (165.2, 159.6)
- SW1, SW10, SW11, SW12, SW13, SW14, SW15, SW16, SW17, SW18, SW19, SW2, SW20, SW21, SW22, SW23, SW24, SW25, SW26, SW27, SW28, SW29, SW3, SW30, SW31, SW32, SW33, SW34, SW35, SW36, SW4, SW5, SW6, SW7, SW8, SW9: footprint benri-projects:GatereonHotswap -> benri-projects:GATEREON_KS-2P02B01-01-a_R
- moved SW2 1.25 mm to (282.0, 119.0)
- moved SW8 1.25 mm to (301.0, 122.2)
- moved SW1 1.10 mm to (278.6, 138.0)
- moved SW7 1.10 mm to (297.6, 141.2)
- moved SW13 0.85 mm to (258.1, 136.5)
- moved SW3 0.85 mm to (260.1, 98.0)
- moved SW9 0.85 mm to (259.1, 117.2)
- moved SW10 0.60 mm to (238.1, 113.2)
- moved SW12 0.60 mm to (199.6, 141.0)
- moved SW14 0.60 mm to (238.1, 132.5)
- moved SW15 0.60 mm to (218.8, 118.5)
- moved SW17 0.60 mm to (218.8, 99.2)
- moved SW18 0.60 mm to (199.6, 102.5)
- moved SW4 0.60 mm to (238.1, 94.0)
- moved SW5 0.60 mm to (218.8, 137.8)
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Connections:
- J1 pad 1: /left/L_3V3 -> /left/L_5V
- J2 pad 1: +3V3 -> 5V
- JP1 pad 2: /left/LTX -> Net-(JP1-B)
- JP2 pad 2: /left/LRX -> Net-(JP2-B)
- JP3 pad 1: +3V3 -> 5V
- JP3 pad 2: /left/L_3V3 -> Net-(JP3-B)
- JP4 pad 2: /left/L_GND -> Net-(JP4-B)
- U1 pad 12: /left/L_3V3 -> unconnected-(U1-3V3-Pad12)
- U1 pad 14: unconnected-(U1-VBUS-Pad14) -> /left/L_5V
- U2 pad 12: +3V3 -> unconnected-(U2-3V3-Pad12)
- U2 pad 14: unconnected-(U2-VBUS-Pad14) -> 5V
Routing:
- net /left/L_3V3: track 37.5 -> 0.00 mm, vias 1 -> 0
- net /left/L_5V: track 0.00 -> 35.8 mm, vias 0 -> 2
- net 5V: track 0.00 -> 30.0 mm
- net +3V3: track 24.6 -> 0.00 mm
- net /left/L_GND: track 13.1 -> 0.00 mm, vias 1 -> 0
- net Net-(JP4-B): track 0.00 -> 12.3 mm
- net Net-(JP3-B): track 0.00 -> 11.8 mm
- net Net-(JP2-B): track 0.00 -> 11.6 mm
- net Net-(JP1-B): track 0.00 -> 11.5 mm
- net /left/column_1: track 107.7 -> 98.2 mm, vias 0 -> 1
- net /left/LTX: track 29.3 -> 21.2 mm, vias 1 -> 0
- net /left/LRX: track 33.9 -> 27.6 mm, vias 1 -> 0
- net /left/row_1: track 48.7 -> 53.9 mm, vias 0 -> 3
- net /left/row_2: track 60.1 -> 65.0 mm, vias 0 -> 3
- net Net-(D16-A): track 15.3 -> 18.7 mm
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Other:
- board size 289.8 x 97.8 mm -> 289.7 x 97.5 mm
- rule pad_to_mask_clearance: 0 -> 0.1

Commit message: Touchups and name: Logos
Parts:
- U1, U2: footprint Seeed Studio XIAO Series Library:XIAO-RP2040-DIP -> benri-projects:SEEED_XIAO-RP2040_T-DIP
- moved U2 0.98 mm to (156.3, 103.0)
- moved U1 0.98 mm to (179.3, 103.0)
Routing:
- net /right/column_2: track 128.4 -> 126.1 mm
- net /right/row_2: track 39.7 -> 41.0 mm
- net /right/RRX: track 24.0 -> 25.3 mm
- net 5V: track 30.0 -> 31.3 mm
- net /left/row_3: track 60.3 -> 61.5 mm
- net /left/row_2: track 65.0 -> 66.2 mm
- net /left/column_2: track 130.4 -> 131.5 mm
- net /left/row_1: track 53.9 -> 55.1 mm
- net /right/column_1: track 87.8 -> 88.9 mm
- net /left/LTX: track 21.2 -> 22.2 mm
- net /left/column_1: track 98.2 -> 99.2 mm
- net /left/column_5: track 187.5 -> 186.5 mm
- net /right/row_4: track 47.6 -> 48.6 mm
- net /left/L_5V: track 35.8 -> 36.8 mm
- net /left/column_3: track 95.3 -> 94.4 mm
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Other:
- board text added: "LOGOS_36_L"
- board text added: "LOGOS_36_R"

Commit message: Base and plate, updates to library, fix diode footprint and symmetry
Parts:
- moved REF** 5.00 mm to (45.5, 134.2)
- moved REF** 5.00 mm to (290.1, 134.2)
- moved SW1 5.00 mm to (278.6, 143.0)
- moved SW2 5.00 mm to (282.0, 124.0)
- moved SW23 5.00 mm to (53.6, 124.0)
- moved SW24 5.00 mm to (57.0, 143.0)
- moved SW29 5.00 mm to (34.6, 127.2)
- moved SW30 5.00 mm to (38.0, 146.2)
- moved SW7 5.00 mm to (297.6, 146.2)
- moved SW8 5.00 mm to (301.0, 127.2)
Routing:
- net /left/column_5: track 186.5 -> 193.2 mm
- net Net-(D30-A): track 109.7 -> 114.1 mm
- net Net-(D29-A): track 114.3 -> 118.4 mm
- net /right/column_5: track 218.0 -> 221.0 mm
- net Net-(D24-A): track 91.0 -> 88.6 mm
- net Net-(D7-A): track 126.6 -> 129.0 mm
- net Net-(D23-A): track 101.8 -> 103.9 mm
- net Net-(D2-A): track 115.2 -> 117.3 mm
- net Net-(D8-A): track 136.2 -> 137.8 mm
Other:
- outline, holes or cut-outs redrawn
- board text added: "LOGOS"

Commit message: Through hole layout
Parts:
- removed ? (x6): , 
- removed JP1, JP2, JP3, JP4, JP5, JP6, JP7, JP8: SolderJumper_2_Open, Jumper:SolderJumper-2_P1.3mm_Open_RoundedPad1.0x1.5mm
- removed the REF** at (165.0, 124.8)
- removed the REF** at (170.7, 124.8)
- D1, D10, D11, D12, D13, D14, D15, D16, D17, D18, D19, D2, D20, D21, D22, D23, D24, D25, D26, D27, D28, D29, D3, D30, D31, D32, D33, D34, D35, D36, D4, D5, D6, D7, D8, D9: footprint benri-projects:DIODES_SOD232_R -> benri-projects:GENERIC_DO-35_A
- J1, J2: footprint benri-projects:TENSILITY_54-00176_R -> benri-projects:JST_SM04B-SR_R
- moved SW18 94.0 mm to (231.2, 191.0), turned to -160 degrees
- moved SW17 92.2 mm to (251.3, 185.5), turned to -170 degrees
- moved SW29 80.2 mm to (104.3, 167.0)
- moved D18 74.4 mm to (231.5, 175.7)
- moved D17 71.1 mm to (231.5, 173.5)
- moved SW1 70.2 mm to (348.3, 151.2)
- moved SW11 65.0 mm to (266.1, 142.5), turned to 180 degrees
- moved SW15 64.1 mm to (266.1, 161.8)
- moved D29 63.9 mm to (200.5, 169.8)
- moved D23 63.5 mm to (200.5, 159.2)
- moved SW16 63.1 mm to (246.9, 165.0), turned to 180 degrees
- moved J2 60.9 mm to (221.3, 141.6)
- moved D35 58.9 mm to (200.5, 176.2)
- moved D36 58.9 mm to (200.5, 174.1)
- moved D30 58.8 mm to (200.5, 172.0)
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Connections:
- J1 pad 1: /left/L_5V -> /right/R_GND
- J1 pad 2: /left/L_GND -> /right/RTX
- J1 pad 3: /left/LTX -> /right/RRX
- J1 pad 4: /left/LRX -> /right/R_5V
- J2 pad 1: 5V -> /left/L_5V
- J2 pad 2: GND -> /left/LTX
- J2 pad 3: /right/RTX -> /left/LRX
- J2 pad 4: /right/RRX -> /left/L_GND
- U2 pad 13: GND -> /right/R_GND
- U2 pad 14: 5V -> /right/R_5V
Routing:
- net /left/L_5V: track 36.8 -> 0.00 mm, vias 2 -> 0
- net 5V: track 31.3 -> 0.00 mm
- net Net-(D17-A): track 54.6 -> 25.7 mm
- net /left/LRX: track 27.7 -> 0.00 mm
- net Net-(D8-A): track 137.8 -> 110.8 mm
- net Net-(D11-A): track 23.0 -> 49.8 mm
- net /right/RRX: track 25.3 -> 0.00 mm
- net /right/RTX: track 24.7 -> 0.00 mm
- net Net-(D1-A): track 106.8 -> 131.1 mm
- net Net-(D29-A): track 118.4 -> 94.6 mm
- net Net-(D18-A): track 31.8 -> 8.67 mm
- net /left/LTX: track 22.2 -> 0.00 mm
- net Net-(D23-A): track 103.9 -> 122.8 mm
- net /right/row_4: track 48.6 -> 34.2 mm, vias 0 -> 1
- net /left/row_2: track 66.2 -> 52.0 mm, vias 3 -> 0
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- added copper zone on B.Cu, net /right/R_GND
- added copper zone on F.Cu, net /right/R_GND
- removed copper zone on B.Cu, net GND
- removed copper zone on F.Cu, net GND
Other:
- outline, holes or cut-outs redrawn
